File: hardware/esp8266-midi.sch (KiCad schematic (older format))
At the start: 20 parts, among them J1 MIDI in, J2 MIDI out, J3 TTL-232R-3V3 connector, J4 Bat+, J5 Bat-, U1 ESP-12E, U2 6N138, U3 LD1117S50TR_SOT223

Commit message: Kicad5: schematic after converting to kicad5, no other changes
Parts:
- C2, C3: symbol C-RESCUE-esp8266-midi -> esp8266-midi-rescue:C-RESCUE-esp8266-midi
- C4: symbol CP -> device:CP
- D1: symbol D -> device:D
- J1, J2: symbol DIN-5_180degree -> Connector1:DIN-5_180degree
- J3: symbol Conn_01x06 -> Connector1:Conn_01x06
- J4, J5: symbol Conn_01x01_Male -> Connector1:Conn_01x01_Male
- R1, R2, R4, R5, R7: symbol R-RESCUE-esp8266-midi -> esp8266-midi-rescue:R-RESCUE-esp8266-midi
- R3, R6, R8: symbol R -> pspice1:R
- U1: symbol ESP-12E -> rfcom:ESP-12E
- U2: symbol 6N138 -> esp8266-midi-rescue:6N138
- U3: symbol LD1117S50TR_SOT223 -> regul:LD1117S50TR_SOT223
Changed lines of the file:
@@
-EESchema Schematic File Version 2
-LIBS:esp8266-midi-rescue
-LIBS:zetex
-LIBS:xilinx
-LIBS:xilinx-virtex7
-LIBS:xilinx-virtex6
-LIBS:xilinx-virtex5
-LIBS:xilinx-spartan6
-LIBS:xilinx-kintex7
-LIBS:xilinx-artix7
-LIBS:wiznet
-LIBS:video
-LIBS:triac_thyristor
-LIBS:texas
-LIBS:supertex
-LIBS:siliconi
-LIBS:silabs
-LIBS:sensors
-LIBS:rfcom
-LIBS:regul
-LIBS:references
-LIBS:pspice
-LIBS:powerint
-LIBS:power
-LIBS:philips
-LIBS:opto
-LIBS:onsemi
-LIBS:nxp
-LIBS:nordicsemi
-LIBS:motorola
-LIBS:motor_drivers
-LIBS:modules
-LIBS:microcontrollers
-LIBS:microchip
-LIBS:memory
-LIBS:maxim
-LIBS:logic_programmable
-LIBS:linear
-LIBS:ir
-LIBS:intersil
-LIBS:interface
-LIBS:intel
-LIBS:infineon
-LIBS:hc11
-LIBS:gennum
-LIBS:ftdi
-LIBS:elec-unifil
-LIBS:dsp
-LIBS:driver_gate
-LIBS:digital-audio
-LIBS:device
-LIBS:dc-dc
-LIBS:cypress
-LIBS:contrib
-LIBS:brooktre
-LIBS:bbd
-LIBS:audio
-LIBS:atmel
-LIBS:analog_switches
-LIBS:analog_devices
-LIBS:adc-dac
-LIBS:ac-dc
-LIBS:Zilog
-LIBS:Xicor
-LIBS:Worldsemi
-LIBS:Valve
-LIBS:Transistor
-LIBS:Transformer
-LIBS:Switch
-LIBS:Sensor_Humidity
-LIBS:Sensor_Current
-LIBS:Relay
-LIBS:RF_Bluetooth
-LIBS:RFSolutions
-LIBS:Power_Management
-LIBS:Oscillators
-LIBS:Motor
-LIBS:Mechanical
-LIBS:MCU_Texas_MSP430
-LIBS:MCU_ST_STM8
-LIBS:MCU_ST_STM32
-LIBS:MCU_Parallax
-LIBS:MCU_NXP_S08
-LIBS:MCU_NXP_LPC
-LIBS:MCU_NXP_Kinetis
-LIBS:MCU_Microchip_PIC32
-LIBS:MCU_Microchip_PIC24
-LIBS:MCU_Microchip_PIC18
-LIBS:MCU_Microchip_PIC16
-LIBS:MCU_Microchip_PIC12
-LIBS:MCU_Microchip_PIC10
-LIBS:Logic_TTL_IEEE
-LIBS:Logic_CMOS_IEEE
-LIBS:Logic_CMOS_4000
-LIBS:Logic_74xx
-LIBS:Logic_74xgxx
-LIBS:Lattice
-LIBS:LEM
-LIBS:LED
-LIBS:Graphic
-LIBS:FPGA_Actel
-LIBS:Espressif
-LIBS:ESD_Protection
-LIBS:Display
-LIBS:Diode
-LIBS:Decawave
-LIBS:DSP_Microchip_DSPIC33
-LIBS:Connector
-LIBS:Bosch
-LIBS:Battery_Management
-LIBS:Altera
+EESchema Schematic File Version 4
 LIBS:esp8266-midi-cache
-EELAYER 25 0
+EELAYER 26 0
 EELAYER END
 $Descr A4 11693 8268
@@
 $EndDescr
 $Comp
-L DIN-5_180degree J2
+L Connector1:DIN-5_180degree J2
 U 1 1 5AA0E52B
 P 7500 5200
@@
 $EndComp
 $Comp
-L DIN-5_180degree J1
+L Connector1:DIN-5_180degree J1
 U 1 1 5AA0E5AD
 P 8600 3250
@@
 $EndComp
 $Comp
-L GND #PWR01
+L power1:GND #PWR01
 U 1 1 5AA0E6C2
 P 7300 4700
@@
 $EndComp
 $Comp
-L +3.3V #PWR02
+L power1:+3.3V #PWR02
 U 1 1 5AA0E7A4
 P 8300 5100
@@
 $EndComp
 $Comp
-L R-RESCUE-esp8266-midi R2
+L esp8266-midi-rescue:R-RESCUE-esp8266-midi R2
 U 1 1 5AA0E7F1
 P 8050 5100
@@
 $EndComp
 $Comp
-L R-RESCUE-esp8266-midi R5
+L esp8266-midi-rescue:R-RESCUE-esp8266-midi R5
 U 1 1 5AA0E839
 P 6950 5100
@@
 $EndComp
 $Comp
-L 6N138 U2
+L esp8266-midi-rescue:6N138 U2
 U 1 1 5AA1AD61
 P 7700 3500
@@
 $EndComp
 $Comp
-L D D1
+L device:D D1
 U 1 1 5AA1AFB6
 P 8150 3500
@@
 $EndComp
 $Comp
-L R-RESCUE-esp8266-midi R1
+L esp8266-midi-rescue:R-RESCUE-esp8266-midi R1
 U 1 1 5AA1B0FD
 P 8600 3750
@@
 $EndComp
 $Comp
-L R-RESCUE-esp8266-midi R4
+L esp8266-midi-rescue:R-RESCUE-esp8266-midi R4
 U 1 1 5AA1C352
 P 7250 3450
@@
 $EndComp
 $Comp
-L +3.3V #PWR03
+L power1:+3.3V #PWR03
 U 1 1 5AA1C85B
 P 7350 3100
@@
 $EndComp
 $Comp
-L GND #PWR04
+L power1:GND #PWR04
 U 1 1 5AA1CB1B
 P 7350 3800
@@
 $EndComp
 $Comp
-L GND #PWR05
+L power1:GND #PWR05
 U 1 1 5AA1FC3D
 P 5650 4400
@@
 NoConn ~ 8900 3250
 $Comp
-L LD1117S50TR_SOT223 U3
+L regul:LD1117S50TR_SOT223 U3
 U 1 1 5AA2FC6F
 P 5450 1850
@@
 $EndComp
 $Comp
-L CP C4
+L device:CP C4
 U 1 1 5AA30545
 P 6200 2100
@@
 $EndComp
 $Comp
-L C-RESCUE-esp8266-midi C3
+L esp8266-midi-rescue:C-RESCUE-esp8266-midi C3
 U 1 1 5AA305EE
 P 5850 2100
@@
 $EndComp
 $Comp
-L C-RESCUE-esp8266-midi C2
+L esp8266-midi-rescue:C-RESCUE-esp8266-midi C2
 U 1 1 5AA30688
 P 5050 2100
@@
 $EndComp
 $Comp
-L +3.3V #PWR06
+L power1:+3.3V #PWR06
 U 1 1 5AA308D3
 P 6400 1850
@@
 $EndComp
 $Comp
-L GND #PWR07
+L power1:GND #PWR07
 U 1 1 5AA310B5
 P 5450 2450
@@
 $EndComp
 $Comp
-L Conn_01x01_Male J4
+L Connector1:Conn_01x01_Male J4
 U 1 1 5AA3271F
 P 4650 1850
@@
 $EndComp
 $Comp
-L Conn_01x01_Male J5
+L Connector1:Conn_01x01_Male J5
 U 1 1 5AA327AB
 P 4650 2350
@@
 $EndComp
 $Comp
-L R-RESCUE-esp8266-midi R7
+L esp8266-midi-rescue:R-RESCUE-esp8266-midi R7
 U 1 1 5AC28C1B
 P 5350 5000
@@
 NoConn ~ 8600 2950
 $Comp
-L ESP-12E U1
+L rfcom:ESP-12E U1
 U 1 1 5AC3DEE1
 P 4200 4600
@@
 $EndComp
 $Comp
-L GND #PWR08
+L power1:GND #PWR08
 U 1 1 5AC3E798
 P 4200 5800
@@
 $EndComp
 $Comp
-L +3.3V #PWR09
+L power1:+3.3V #PWR09
 U 1 1 5AC3F393
 P 4200 3400
@@
 $EndComp
 $Comp
-L +3.3V #PWR010
+L power1:+3.3V #PWR010
 U 1 1 5AC3FC81
 P 2700 4100
@@
 $EndComp
 $Comp
-L GND #PWR011
+L power1:GND #PWR011
 U 1 1 5AC41342
 P 5600 5100
@@
 NoConn ~ 5100 4300
 $Comp
-L R R6
+L pspice1:R R6
 U 1 1 5B127227
 P 3850 3450
@@
 $EndComp
 $Comp
-L R R8
+L pspice1:R R8
 U 1 1 5B1275B7
 P 4550 3450
@@
 	7050 3450 7050 3700
 Wire Wire Line
-	7050 3700 7450 3700
+	7050 3700 7350 3700
 Wire Wire Line
 	7350 3700 7350 3800
@@
 	6400 3550 7450 3550
 Wire Wire Line
-	5750 1850 6400 1850
+	5750 1850 5850 1850
 Wire Wire Line
 	5850 1850 5850 1950
@@
 Connection ~ 5850 2350
 Wire Wire Line
-	5450 2150 5450 2450
+	5450 2150 5450 2350
 Connection ~ 5450 2350
 Connection ~ 5050 1850
@@
 	4200 5700 4200 5800
 Wire Wire Line
-	4200 3400 4200 3500
+	4200 3400 4200 3450
 Connection ~ 4200 3450
 Wire Wire Line
@@
 	7350 3300 7450 3300
 Wire Wire Line
-	4100 3450 4300 3450
+	4100 3450 4200 3450
 Wire Wire Line
 	4800 3450 5150 3450
@@
 	5150 3450 5150 3800
 Wire Wire Line
-	5100 3800 5750 3800
-Wire Wire Line
-	3600 3450 3250 3450
+	5100 3800 5150 3800
+Wire Wire Line
+	3600 3450 3550 3450
 Wire Wire Line
 	3250 3450 3250 3800
@@
 	3250 3800 3300 3800
 $Comp
-L R R3
+L pspice1:R R3
 U 1 1 5B12802D
 P 3000 4000
@@
 	2700 4000 2700 4100
 $Comp
-L Conn_01x06 J3
+L Connector1:Conn_01x06 J3
 U 1 1 5AA1FA8A
 P 6000 4500
@@
 Connection ~ 3550 3450
 Wire Wire Line
-	4850 1850 5150 1850
-Wire Wire Line
-	4850 2350 6200 2350
+	4850 1850 5050 1850
+Wire Wire Line
+	4850 2350 5050 2350
+Wire Wire Line
+	7350 3700 7450 3700
+Wire Wire Line
+	5850 1850 6200 1850
+Wire Wire Line
+	6200 1850 6400 1850
+Wire Wire Line
+	5850 2350 6200 2350
+Wire Wire Line
+	5450 2350 5450 2450
+Wire Wire Line
+	5450 2350 5850 2350
+Wire Wire Line
+	5050 1850 5150 1850
+Wire Wire Line
+	5050 2350 5450 2350
+Wire Wire Line
+	4200 3450 4200 3500
+Wire Wire Line
+	4200 3450 4300 3450
+Wire Wire Line
+	5150 3800 5750 3800
+Wire Wire Line
+	3550 3450 3250 3450
 $EndSCHEMATC
