File: hardware/esp8266-midi.kicad_pcb (KiCad board)
At the start: 2 copper layers, 75 x 82 mm, 31 parts, among them J1 MIDI in, J2 MIDI out, J3 TTL-232R-3V3 connector, J4 Bat+, J5 Bat-, J6 MIDI through, J7 Debug serial out, U1 ESP-12E, U2 6N138, U3 LD1117S50TR_SOT223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

Commit message: Use alternative uart0 pins for midi i/o
uart0 pushes bunch of rubbish messages on boot up. This means some pretty random
messages on the midi out port. To fix this midi i/o uses alternative uart0 pins
which can be enabled after microcontroller is booted by calling 'Serial.swap()'.

Alternative TX pin needs to be pulled down during boot, but a connected midi
instrument pull it up. Therefore the buffering using the same dual nand
(74LVC2G14) as for the midi through port.
Parts:
- added C5: 100nF, Capacitors_SMD:C_0805_HandSoldering, F.Cu at (168.0, 99.0)
- added U5: 74LVC2G14, TO_SOT_Packages_SMD:SOT-23-6_Handsoldering, F.Cu at (171.0, 99.0)
- moved C4 10.7 mm to (132.0, 86.5), turned to 180 degrees
- moved J5 9.04 mm to (127.1, 93.7), turned to 270 degrees
- moved U3 8.68 mm to (143.0, 90.0)
- moved C2 7.43 mm to (138.5, 90.2)
- moved J4 1.96 mm to (132.2, 93.7), turned to 270 degrees
- moved R7 1.50 mm to (151.0, 85.0)
Connections:
- R5 pad 1: UART0_TXD -> Net-(R5-Pad1)
- R7 pad 1: Net-(R7-Pad1) -> GND
- R7 pad 2: GND -> UART0_ALT_TXD
- U1 pad 16: Net-(R7-Pad1) -> UART0_ALT_TXD
- U1 pad 7: (no net) -> UART0_ALT_RXD
- U2 pad 6: UART0_RXD -> UART0_ALT_RXD
- U4 pad 1: UART0_RXD -> UART0_ALT_RXD
Routing:
- net UART0_ALT_RXD: track 0.00 -> 71.0 mm, vias 0 -> 3
- net UART0_RXD: track 95.6 -> 34.8 mm, vias 3 -> 1
- net UART0_TXD: track 79.4 -> 35.1 mm
- net UART0_ALT_TXD: track 0.00 -> 33.7 mm
- net UART1_TXD: track 31.0 -> 17.9 mm, vias 1 -> 0
- net Net-(R7-Pad1): track 9.01 -> 0.00 mm
- net Net-(C2-Pad1): track 6.43 -> 11.5 mm
- net Net-(U5-Pad3): track 0.00 -> 4.06 mm
- net Net-(R5-Pad1): track 0.00 -> 2.75 mm
- net GND: track 1.15 -> 3.30 mm, vias 2 -> 6
- net VCC: track 119.6 -> 119.0 mm, vias 7 -> 4
